File: HS-TARGET_001/HS-TARGET_001.sch (KiCad schematic (older format))
At the start: 39 parts

Commit message: ・HS-TARGET001更新
Parts:
- removed Y?: Crystal, symbol Device:Crystal_GND2
- added J5: dry_cell, Connector_PinHeader_2.54mm:PinHeader_1x02_P2.54mm_Vertical, symbol Connector_Generic:Conn_01x02
- added JP3: Jumper, Connector_PinHeader_2.54mm:PinHeader_1x02_P2.54mm_Vertical, symbol Device:Jumper
- added U6: AE-XCL102D503CR-G, hotsprings-footprints:AE-XCL102D503CR-G, symbol HotSprings:AE-XCL102D503CR-G
- added Y1: Crystal, Crystal:Crystal_HC49-4H_Vertical, symbol Device:Crystal
- C1, C2, C3, C5, C6: renamed from C?; footprint (none) -> Capacitor_SMD:C_1206_3216Metric
- C4, C7: renamed from C?; footprint (none) -> Capacitor_THT:CP_Radial_D6.3mm_P2.50mm
- D1: renamed from D?; footprint (none) -> LED_THT:LED_D5.0mm
- D2: renamed from D?; footprint (none) -> Connector_PinHeader_2.54mm:PinHeader_1x04_P2.54mm_Vertical
- J2: renamed from J?; footprint (none) -> Connector_PinHeader_2.54mm:PinHeader_1x02_P2.54mm_Vertical
- J3: renamed from J?; footprint (none) -> Connector_PinHeader_2.54mm:PinHeader_2x03_P2.54mm_Vertical
- J4: renamed from J?; footprint (none) -> Connector_PinHeader_2.54mm:PinHeader_1x06_P2.54mm_Vertical
- JP1, JP2: renamed from JP?; footprint (none) -> Connector_PinHeader_2.54mm:PinHeader_1x03_P2.54mm_Vertical
- LS1: renamed from LS?; footprint (none) -> Connector_PinHeader_2.54mm:PinHeader_1x02_P2.54mm_Vertical
- Q1, Q2, Q3: renamed from Q?; footprint (none) -> digikey-footprints:SOT-23W
- R1, R10, R2, R3, R4, R5, R6, R7, R8, R9: renamed from R?; footprint (none) -> Resistor_THT:R_Axial_DIN0204_L3.6mm_D1.6mm_P7.62mm_Horizontal
- SW1: renamed from SW?; footprint (none) -> Button_Switch_THT:SW_TH_Tactile_Omron_B3F-10xx
- SW2: renamed from SW?; footprint (none) -> Button_Switch_THT:SW_DIP_SPSTx04_Slide_6.7x11.72mm_W7.62mm_P2.54mm_LowProfile
- U3: renamed from U?; footprint (none) -> hotsprings-footprints:DFPlayer-MINI
- U4: renamed from U?; footprint (none) -> hotsprings-footprints:TWELITE-DIP
- gave numbers to parts that had none: 6
Connections:
- net GND: now also SW2.5, SW2.6, SW2.7, SW2.8
- net at U2.10 (XTAL2/PB7): now also Y1.2
- net at U2.9 (XTAL1/PB6): now also Y1.1
- net at C4.1, C5.1, F1.2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: now also JP3.2
- new net: J5.2 (Pin_2), U6.4 (IN)
- new net: J5.1 (Pin_1), U6.5 (GND)
- new net: JP3.1, U6.6 (OUT)

Commit message: ・HS-TARGET001基盤作図開始
Parts:
- added JP4: Mode_Switch, Connector_PinHeader_2.54mm:PinHeader_2x01_P2.54mm_Vertical, symbol Device:Jumper
- F1: footprint (none) -> Diode_THT:D_DO-41_SOD81_P10.16mm_Horizontal
- U5: footprint Converter_DCDC:Converter_DCDC_RECOM_R-78E-0.5_THT -> Package_TO_SOT_SMD:TO-252-2
Connections:
- net GND: now also JP4.2
- net MODE_SW: now reaches U2.14 (PB0)
- net MODE_SW: now also JP4.1
Changed lines of the file:
@@
 F 0 "U5" H 8950 5992 50  0000 C CNN
 F 1 "R-781.8-1.0" H 8950 5901 50  0000 C CNN
-F 2 "Converter_DCDC:Converter_DCDC_RECOM_R-78E-0.5_THT" H 9000 5500 50  0001 L CIN
+F 2 "Package_TO_SOT_SMD:TO-252-2" H 9000 5500 50  0001 L CIN
 F 3 "https://www.recom-power.com/pdf/Innoline/R-78xx-1.0.pdf" H 8950 5750 50  0001 C CNN
 	1    8950 5750
@@
 F 0 "F1" H 7650 5935 50  0000 C CNN
 F 1 "Fuse_Small" H 7650 5844 50  0000 C CNN
-F 2 "" H 7650 5750 50  0001 C CNN
+F 2 "Diode_THT:D_DO-41_SOD81_P10.16mm_Horizontal" H 7650 5750 50  0001 C CNN
 F 3 "~" H 7650 5750 50  0001 C CNN
 	1    7650 5750
@@
 Wire Wire Line
 	7900 5300 7700 5300
+$Comp
+L Device:Jumper JP4
+U 1 1 5D72B739
+P 7500 4350
+F 0 "JP4" H 7500 4614 50  0000 C CNN
+F 1 "Mode_Switch" H 7500 4523 50  0000 C CNN
+F 2 "Connector_PinHeader_2.54mm:PinHeader_2x01_P2.54mm_Vertical" H 7500 4350 50  0001 C CNN
+F 3 "~" H 7500 4350 50  0001 C CNN
+	1    7500 4350
+	1    0    0    -1
+$EndComp
+Text GLabel 2300 1650 2    50   Input ~ 0
+MODE_SW
+Text GLabel 7200 4350 0    50   Input ~ 0
+MODE_SW
+Text GLabel 7800 4350 2    50   Input ~ 0
+GND
 $EndSCHEMATC

Commit message: ・HS-TARGET001基盤修正 ・HS-TAGLED001 開始
Parts:
- removed JP3: Jumper, Connector_PinHeader_2.54mm:PinHeader_1x02_P2.54mm_Vertical, symbol Device:Jumper
- SW1: footprint Button_Switch_THT:SW_TH_Tactile_Omron_B3F-10xx -> digikey-footprints:Switch_Tactile_THT_6x6mm
Connections:
- net at C4.1, C5.1, F1.2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: now also U6.6 (OUT)
Changed lines of the file:
@@
 F 0 "SW1" H 3800 3385 50  0000 C CNN
 F 1 "RESET" H 3800 3294 50  0000 C CNN
-F 2 "Button_Switch_THT:SW_TH_Tactile_Omron_B3F-10xx" H 3800 3150 50  0001 C CNN
+F 2 "digikey-footprints:Switch_Tactile_THT_6x6mm" H 3800 3150 50  0001 C CNN
 F 3 "~" H 3800 3150 50  0001 C CNN
 	1    3800 3150
@@
 $EndComp
 Connection ~ 7950 5750
-Wire Wire Line
-	7750 5750 7900 5750
 $Comp
 L HotSprings:AE-XCL102D503CR-G U6
@@
 	1    0    0    -1
 $EndComp
-$Comp
-L Device:Jumper JP3
-U 1 1 5D7BA38C
-P 8200 5200
-F 0 "JP3" V 8154 5327 50  0000 L CNN
-F 1 "Jumper" V 8245 5327 50  0000 L CNN
-F 2 "Connector_PinHeader_2.54mm:PinHeader_1x02_P2.54mm_Vertical" H 8200 5200 50  0001 C CNN
-F 3 "~" H 8200 5200 50  0001 C CNN
-	1    8200 5200
-	0    1    1    0
-$EndComp
 Wire Wire Line
 	7850 4900 8200 4900
-Wire Wire Line
-	8200 5500 7900 5500
-Wire Wire Line
-	7900 5500 7900 5750
-Connection ~ 7900 5750
-Wire Wire Line
-	7900 5750 7950 5750
 $Comp
 L Connector_Generic:Conn_01x02 J5
@@
 	7850 5000 8050 5000
 Wire Wire Line
-	8050 5000 8050 5400
-Wire Wire Line
-	8050 5400 7700 5400
-Wire Wire Line
 	7850 5100 7900 5100
-Wire Wire Line
-	7900 5100 7900 5300
-Wire Wire Line
-	7900 5300 7700 5300
 $Comp
 L Device:Jumper JP4
@@
 Text GLabel 7800 4350 2    50   Input ~ 0
 GND
+Wire Wire Line
+	8200 4900 8200 5500
+Wire Wire Line
+	7900 5300 7700 5300
+Wire Wire Line
+	7900 5100 7900 5300
+Wire Wire Line
+	8050 5400 7700 5400
+Wire Wire Line
+	8050 5000 8050 5400
+Wire Wire Line
+	7750 5750 7950 5750
+Wire Wire Line
+	8200 5500 7950 5500
+Wire Wire Line
+	7950 5500 7950 5750
 $EndSCHEMATC
