File: TWE-TARGET/TWE-TARGET.sch (KiCad schematic (older format))
At the start: 27 parts, among them J1 5V_Serial, J2 B2B-PH-K-S_LF__SN_, J3 Conn_01x07, J4 PROG, J5 Conn_02x06_Counter_Clockwise, Q1 Q_NMOS_GSD, Q2 Q_NMOS_GSD, Q3 Q_NMOS_GSD, SW1 SW_DPST_x2, U1 TSOP59540TR1, U2 ATmega328P-PU, U3 TWE-L-WX, U5 R-781.8-1.0, Y1 Crystal_GND2

Commit message: ・TWEーTARGET更新
Parts:
- R10, R8, R9: value 3.3k -> 1.0k
Changed lines of the file:
@@
 P 4850 3950
 F 0 "R8" H 4918 3996 50  0000 L CNN
-F 1 "3.3k" H 4918 3905 50  0000 L CNN
+F 1 "1.0k" H 4918 3905 50  0000 L CNN
 F 2 "Capacitor_SMD:C_1206_3216Metric" V 4890 3940 50  0001 C CNN
 F 3 "~" H 4850 3950 50  0001 C CNN
@@
 P 5050 3950
 F 0 "R9" H 5118 3996 50  0000 L CNN
-F 1 "3.3k" H 5118 3905 50  0000 L CNN
+F 1 "1.0k" H 5118 3905 50  0000 L CNN
 F 2 "Capacitor_SMD:C_1206_3216Metric" V 5090 3940 50  0001 C CNN
 F 3 "~" H 5050 3950 50  0001 C CNN
@@
 P 5250 3950
 F 0 "R10" H 5318 3996 50  0000 L CNN
-F 1 "3.3k" H 5318 3905 50  0000 L CNN
+F 1 "1.0k" H 5318 3905 50  0000 L CNN
 F 2 "Capacitor_SMD:C_1206_3216Metric" V 5290 3940 50  0001 C CNN
 F 3 "~" H 5250 3950 50  0001 C CNN
